Commit message: enabled collision detection on the camera mount

File: xarm_description/urdf/common/common.link.xacro (robot description, xacro)
@@ -38,9 +38,9 @@
     </visual>
   </xacro:macro>
-  <xacro:macro name="common_link_collision" params="mesh_filename add_mesh_suffix:=true origin_xyz:='0 0 0' origin_rpy:='0 0 0'">
+  <xacro:macro name="common_link_collision" params="mesh_filename add_mesh_suffix:=true origin_xyz:='0 0 0' origin_rpy:='0 0 0' mesh_scale:='1 1 1'">
     <collision>
       <geometry>
         <xacro:if value="${add_mesh_suffix}">
-          <mesh filename="${mesh_path}/${mesh_filename}.${mesh_suffix}"/>
+          <mesh filename="${mesh_path}/${mesh_filename}.${mesh_suffix}" scale="${mesh_scale}"/>
         </xacro:if>
         <xacro:unless value="${add_mesh_suffix}">

File: xarm_description/urdf/mount/gelsight_realsense_d405.urdf.xacro (robot description, xacro)
@@ -11,8 +11,9 @@
         origin_rpy="${M_PI/2} 0 0"
         material_name="${prefix}Silver" />
-      <!-- <xacro:common_link_collision
-        mesh_filename="camera/realsense/collision/d435_with_cam_stand"
+      <xacro:common_link_collision
+        mesh_filename="mount/collision/gelsight_realsense_d405"
+        mesh_scale="0.001 0.001 0.001"
         origin_xyz="0 0 0"
-        origin_rpy="0 0 0" /> -->
+        origin_rpy="${M_PI/2} 0 0" />
     </link>
     <xacro:if value="${add_d405_links}">
